File: pcb/server/server.kicad_pcb (KiCad board)
At the start: 2 copper layers, 83.6 x 66.2 mm, 15 parts, among them IC1 ATMEGA328P-P, P1 nRF24L01, P3 CONN_01X02, Q1 BC548, U1 LM2931AZ-3.3/5.0, Y1 8Mhz

Commit message: test
Parts:
- C1, C3: value 22n -> 22p
- U1: value LM2931AZ-3.3/5.0 -> HT7333
Changed lines of the file:
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@@
       (effects (font (size 1 1) (thickness 0.15)))
     )
-    (fp_text value 22n (at 2.09 2.37) (layer F.Fab)
+    (fp_text value 22p (at 2.09 2.37) (layer F.Fab)
       (effects (font (size 1 1) (thickness 0.15)))
     )
@@
       (effects (font (size 1 1) (thickness 0.15)))
     )
-    (fp_text value 22n (at 2.16 -2.32) (layer F.Fab)
+    (fp_text value 22p (at 2.16 -2.32) (layer F.Fab)
       (effects (font (size 1 1) (thickness 0.15)))
     )
@@
       (effects (font (size 1 1) (thickness 0.15)))
     )
-    (fp_text value LM2931AZ-3.3/5.0 (at -2.34 -3.49 360) (layer F.Fab)
+    (fp_text value HT7333 (at -1.48 -4.49 360) (layer F.Fab)
       (effects (font (size 1 1) (thickness 0.15)))
     )
@@
   (gr_line (start 84.72 40.89) (end 168.29 40.89) (angle 90) (layer Edge.Cuts) (width 0.15))
   (segment (start 102.77 58.7715) (end 102.5085 58.51) (width 0.25) (layer B.Cu) (net 0))
-  (segment (start 127.97 73.2) (end 125.23 73.2) (width 0.35) (layer B.Cu) (net 1) (status 400000))
-  (segment (start 120.31 80.897857) (end 122.652143 83.24) (width 0.35) (layer B.Cu) (net 1) (status 800000))
+  (segment (start 127.97 73.2) (end 125.23 73.2) (width 0.35) (layer B.Cu) (net 1))
+  (segment (start 120.31 80.897857) (end 122.652143 83.24) (width 0.35) (layer B.Cu) (net 1))
   (segment (start 120.31 75.66) (end 120.31 80.897857) (width 0.35) (layer B.Cu) (net 1))
   (segment (start 121.65 74.32) (end 120.31 75.66) (width 0.35) (layer B.Cu) (net 1))
   (segment (start 124.11 74.32) (end 121.65 74.32) (width 0.35) (layer B.Cu) (net 1))
   (segment (start 125.23 73.2) (end 124.11 74.32) (width 0.35) (layer B.Cu) (net 1))
-  (segment (start 101.76 71.19) (end 102.15 71.19) (width 0.35) (layer B.Cu) (net 1) (status C00000))
-  (segment (start 102.15 71.19) (end 106.76 66.58) (width 0.35) (layer B.Cu) (net 1) (status 400000))
-  (segment (start 141.15 58.34) (end 141.15 76.22) (width 0.35) (layer B.Cu) (net 1) (status 800000))
+  (segment (start 101.76 71.19) (end 102.15 71.19) (width 0.35) (layer B.Cu) (net 1))
+  (segment (start 102.15 71.19) (end 106.76 66.58) (width 0.35) (layer B.Cu) (net 1))
+  (segment (start 141.15 58.34) (end 141.15 76.22) (width 0.35) (layer B.Cu) (net 1))
   (segment (start 135.06 52.25) (end 141.15 58.34) (width 0.35) (layer B.Cu) (net 1))
   (segment (start 107.34 52.25) (end 135.06 52.25) (width 0.35) (layer B.Cu) (net 1))
   (segment (start 106.76 52.83) (end 107.34 52.25) (width 0.35) (layer B.Cu) (net 1))
   (segment (start 106.76 66.58) (end 106.76 52.83) (width 0.35) (layer B.Cu) (net 1))
-  (segment (start 141.15 76.22) (end 149.37 76.22) (width 0.35) (layer B.Cu) (net 1) (status 400000))
-  (segment (start 151.91 90.36) (end 146.99 95.28) (width 0.35) (layer B.Cu) (net 1) (status 800000))
+  (segment (start 141.15 76.22) (end 149.37 76.22) (width 0.35) (layer B.Cu) (net 1))
+  (segment (start 151.91 90.36) (end 146.99 95.28) (width 0.35) (layer B.Cu) (net 1))
   (segment (start 151.91 78.76) (end 151.91 90.36) (width 0.35) (layer B.Cu) (net 1))
   (segment (start 149.37 76.22) (end 151.91 78.76) (width 0.35) (layer B.Cu) (net 1))
@@
   (segment (start 126.46 80.75) (end 122.702143 80.75) (width 0.35) (layer B.Cu) (net 10))
   (segment (start 122.702143 80.75) (end 122.652143 80.7) (width 0.35) (layer B.Cu) (net 10))
-  (segment (start 138.02 92.04) (end 138.02 92.33) (width 0.35) (layer B.Cu) (net 11) (status C00000))
-  (segment (start 138.02 92.33) (end 136.75 93.6) (width 0.35) (layer B.Cu) (net 11) (status 400000))
-  (segment (start 106.95 99.91) (end 101.06 94.02) (width 0.35) (layer B.Cu) (net 11) (status 800000))
+  (segment (start 138.02 92.04) (end 138.02 92.33) (width 0.35) (layer B.Cu) (net 11))
+  (segment (start 138.02 92.33) (end 136.75 93.6) (width 0.35) (layer B.Cu) (net 11))
+  (segment (start 106.95 99.91) (end 101.06 94.02) (width 0.35) (layer B.Cu) (net 11))
   (segment (start 135.09 99.91) (end 106.95 99.91) (width 0.35) (layer B.Cu) (net 11))
   (segment (start 136.75 98.25) (end 135.09 99.91) (width 0.35) (layer B.Cu) (net 11))
   (segment (start 136.75 93.6) (end 136.75 98.25) (width 0.35) (layer B.Cu) (net 11))
-  (segment (start 101.11 89.27) (end 101.11 81.88) (width 0.35) (layer B.Cu) (net 11) (status 400000))
-  (segment (start 101.11 81.88) (end 102.44 80.55) (width 0.35) (layer B.Cu) (net 11) (status 800000))
-  (segment (start 101.06 94.02) (end 101.06 89.32) (width 0.35) (layer B.Cu) (net 11) (status C00000))
-  (segment (start 101.06 89.32) (end 101.11 89.27) (width 0.35) (layer B.Cu) (net 11) (status C00000))
+  (segment (start 101.11 89.27) (end 101.11 81.88) (width 0.35) (layer B.Cu) (net 11))
+  (segment (start 101.11 81.88) (end 102.44 80.55) (width 0.35) (layer B.Cu) (net 11))
+  (segment (start 101.06 94.02) (end 101.06 89.32) (width 0.35) (layer B.Cu) (net 11))
+  (segment (start 101.06 89.32) (end 101.11 89.27) (width 0.35) (layer B.Cu) (net 11))
   (segment (start 138.02 92.04) (end 146.43 92.04) (width 0.35) (layer B.Cu) (net 11))
   (segment (start 146.43 92.04) (end 146.99 91.48) (width 0.35) (layer B.Cu) (net 11))
@@
   (segment (start 99.22 71.19) (end 99.22 61.1115) (width 0.35) (layer B.Cu) (net 12))
   (segment (start 99.22 61.1115) (end 99.3115 61.02) (width 0.25) (layer B.Cu) (net 12))
-  (segment (start 109.19 93.72094) (end 103.85906 93.72094) (width 0.35) (layer B.Cu) (net 13) (status C00000))
-  (segment (start 103.85906 93.72094) (end 103.56 94.02) (width 0.25) (layer B.Cu) (net 13) (status C00000))
-  (segment (start 115.032143 85.78) (end 115.032143 86.107857) (width 0.25) (layer B.Cu) (net 13) (status C00000))
-  (segment (start 115.032143 86.107857) (end 109.19 91.95) (width 0.35) (layer B.Cu) (net 13) (status 400000))
-  (segment (start 109.19 91.95) (end 109.19 93.72094) (width 0.35) (layer B.Cu) (net 13) (status 800000))
-  (segment (start 109.19 88.83906) (end 104.04094 88.83906) (width 0.35) (layer B.Cu) (net 14) (status C00000))
-  (segment (start 104.04094 88.83906) (end 103.61 89.27) (width 0.25) (layer B.Cu) (net 14) (status C00000))
-  (segment (start 115.032143 83.24) (end 114.78906 83.24) (width 0.25) (layer B.Cu) (net 14) (status C00000))
-  (segment (start 114.78906 83.24) (end 109.19 88.83906) (width 0.35) (layer B.Cu) (net 14) (status C00000))
+  (segment (start 109.19 93.72094) (end 103.85906 93.72094) (width 0.35) (layer B.Cu) (net 13))
+  (segment (start 103.85906 93.72094) (end 103.56 94.02) (width 0.25) (layer B.Cu) (net 13))
+  (segment (start 115.032143 85.78) (end 115.032143 86.107857) (width 0.25) (layer B.Cu) (net 13))
+  (segment (start 115.032143 86.107857) (end 109.19 91.95) (width 0.35) (layer B.Cu) (net 13))
+  (segment (start 109.19 91.95) (end 109.19 93.72094) (width 0.35) (layer B.Cu) (net 13))
+  (segment (start 109.19 88.83906) (end 104.04094 88.83906) (width 0.35) (layer B.Cu) (net 14))
+  (segment (start 104.04094 88.83906) (end 103.61 89.27) (width 0.25) (layer B.Cu) (net 14))
+  (segment (start 115.032143 83.24) (end 114.78906 83.24) (width 0.25) (layer B.Cu) (net 14))
+  (segment (start 114.78906 83.24) (end 109.19 88.83906) (width 0.35) (layer B.Cu) (net 14))
 )
