File: pcb/sensor21/sensor21.kicad_pcb (KiCad board)
At the start: 2 copper layers, 83.5 x 66.2 mm, 34 parts, among them IC1 ATMEGA8-P, P1 nRF24L01, P2 BME280, P3 CONN_01X02, Q1 BC548, U1 LM2931AZ-3.3/5.0, Y1 8Mhz

Commit message: all works ok
Parts:
- removed 1-REF**, 2-REF**, 3-REF**, 4-REF**, 5-REF**, 6-REF**, 7-REF**, 8-REF**, LB-REF**, LT-REF**, RB-REF**, RT-REF**: 1pin, Connect:1pin
- added C10: 10u, Capacitors_ThroughHole:C_Radial_D5_L11_P2, F.Cu at (155.6, 102.9)
- added C9: 10u, Capacitors_ThroughHole:C_Radial_D5_L11_P2, F.Cu at (121.7, 97.0)
- U1: value LM2931AZ-3.3/5.0 -> HT7333
- moved R6 62.4 mm to (177.1, 86.8), turned to 180 degrees
- moved R5 54.6 mm to (177.1, 90.3), turned to 180 degrees
- moved R3 48.4 mm to (177.0, 102.0)
- moved C1 47.8 mm to (137.1, 120.4)
- moved C4 47.4 mm to (161.7, 106.5), turned to 90 degrees
- moved Q1 42.5 mm to (133.3, 91.8), turned to 270 degrees
- moved C3 42.4 mm to (133.9, 120.4), turned to 180 degrees
- moved P2 41.1 mm to (154.0, 86.9)
- moved R4 40.4 mm to (154.0, 92.2)
- moved C5 39.1 mm to (134.3, 107.4), turned to 0 degrees
- moved U1 38.8 mm to (124.0, 103.0)
- moved C6 38.6 mm to (123.7, 110.7), turned to 180 degrees
- moved C2 37.6 mm to (152.8, 107.6)
- moved R7 37.1 mm to (138.4, 96.7)
- moved IC1 36.5 mm to (142.2, 87.2)
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Connections:
- IC1 pad 11: Net-(IC1-Pad11) -> (no net)
- IC1 pad 12: Net-(IC1-Pad12) -> (no net)
- IC1 pad 14: Net-(IC1-Pad14) -> (no net)
- IC1 pad 2: Net-(IC1-Pad2) -> (no net)
- IC1 pad 23: Net-(IC1-Pad23) -> (no net)
- IC1 pad 26: Net-(IC1-Pad26) -> (no net)
- IC1 pad 3: Net-(IC1-Pad3) -> (no net)
- IC1 pad 4: Net-(IC1-Pad4) -> (no net)
- IC1 pad 6: Net-(IC1-Pad6) -> (no net)
Routing:
- net +3V3: track 317.2 -> 202.6 mm
- net GND: track 311.7 -> 254.4 mm
- net PD7: track 55.5 -> 32.9 mm
- net PC1: track 34.4 -> 22.2 mm
- net PC2: track 41.3 -> 29.6 mm
- net MOSI: track 20.6 -> 10.1 mm
- net CSN: track 22.9 -> 12.7 mm
- net SDA: track 31.9 -> 23.9 mm
- net SCL: track 27.0 -> 21.0 mm
- net Net-(C9-Pad1): track 10.2 -> 15.8 mm
- net Net-(C1-Pad2): track 14.1 -> 19.4 mm
- net SCK: track 14.6 -> 11.2 mm
- net MISO: track 9.66 -> 7.58 mm
- net CE: track 16.8 -> 18.7 mm
- net RESET: track 13.4 -> 11.9 mm
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Other:
- board size 83.5 x 66.2 mm -> 123.1 x 71.8 mm
- net class moje removed
- rule pad_to_mask_clearance: 0.2 -> 0
- board text removed: "Sensor21 v2.2"

Commit message: server side work fine
Other:
- board size 123.1 x 71.8 mm -> 66.3 x 46.8 mm

Commit message: all work well
Parts:
- C2, C4, C5: footprint Capacitors_ThroughHole:C_Disc_D6_P5 -> Capacitors_ThroughHole:C_Disc_D3_P2.5
- U1: footprint TO_SOT_Packages_THT:TO-92_Inline_Narrow_Oval -> TO_SOT_Packages_THT:TO-92_Inline_Wide
- moved C4 3.30 mm to (161.6, 103.2)
- moved C8 2.33 mm to (173.3, 116.6)
- moved C6 2.07 mm to (121.6, 110.8), turned to 0 degrees
- moved C5 1.36 mm to (135.7, 107.5)
- moved C2 1.36 mm to (154.1, 107.6)
- moved U1 1.18 mm to (125.0, 103.6)
- moved P1 0.83 mm to (165.2, 116.5)
Connections:
- IC1 pad 11: (no net) -> Net-(IC1-Pad11)
- IC1 pad 12: (no net) -> Net-(IC1-Pad12)
- IC1 pad 14: (no net) -> Net-(IC1-Pad14)
- IC1 pad 2: (no net) -> Net-(IC1-Pad2)
- IC1 pad 23: (no net) -> Net-(IC1-Pad23)
- IC1 pad 26: (no net) -> Net-(IC1-Pad26)
- IC1 pad 3: (no net) -> Net-(IC1-Pad3)
- IC1 pad 4: (no net) -> Net-(IC1-Pad4)
- IC1 pad 6: (no net) -> Net-(IC1-Pad6)
- U1 pad 1: +3V3 -> GND
- U1 pad 2: GND -> Net-(C9-Pad1)
- U1 pad 3: Net-(C9-Pad1) -> +3V3
Routing:
- net +3V3: track 202.6 -> 237.1 mm
- net CSN: track 12.7 -> 14.9 mm
- net GND: track 254.4 -> 252.4 mm
- net CE: track 18.7 -> 20.6 mm
- net Net-(C2-Pad1): track 4.00 -> 5.07 mm
- net PC2: track 29.6 -> 30.5 mm
- net Net-(C9-Pad1): track 15.8 -> 16.7 mm
- net INT1: track 32.4 -> 33.2 mm
- net MISO: track 7.58 -> 8.41 mm
- net SCK: track 11.2 -> 12.0 mm
- net PD7: track 32.9 -> 33.6 mm
- net MOSI: track 10.1 -> 10.8 mm

Commit message: some mesurements
Parts:
- added C11: 100n, Capacitors_ThroughHole:C_Disc_D3_P2.5, F.Cu at (121.6, 95.8)
- added C12: 100n, Capacitors_ThroughHole:C_Disc_D3_P2.5, F.Cu at (120.9, 112.0)
- moved C6 6.38 mm to (121.1, 117.2)
- moved C9 3.79 mm to (122.0, 100.8)
- moved U1 3.36 mm to (124.8, 107.0)
Routing:
- net GND: track 252.4 -> 270.8 mm
- net +3V3: track 237.1 -> 252.4 mm
- net Net-(C11-Pad1): track 16.7 -> 19.9 mm

Commit message: wip
Parts:
- added REF**: MountingHole_3mm, Mounting_Holes:MountingHole_3mm, F.Cu at (112.6, 83.4)
- added REF**: MountingHole_3mm, Mounting_Holes:MountingHole_3mm, F.Cu at (183.1, 83.5)
- added REF**: MountingHole_3mm, Mounting_Holes:MountingHole_3mm, F.Cu at (182.9, 120.4)
- added REF**: MountingHole_3mm, Mounting_Holes:MountingHole_3mm, F.Cu at (112.5, 120.5)
Routing:
- added copper zone on B.Cu, net GND
Other:
- board size 66.3 x 46.8 mm -> 80.1 x 48 mm
Changed lines of the file:
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@@
     (links 61)
     (no_connects 0)
-    (area 115.289999 77.549999 181.660001 124.440001)
+    (area 106.061474 77.549999 191.540046 126.42626)
     (thickness 1.6)
     (drawings 5)
     (tracks 343)
     (zones 0)
-    (modules 26)
+    (modules 30)
     (nets 28)
   )
@@
     (last_trace_width 0.25)
     (trace_clearance 0.2)
-    (zone_clearance 0.508)
+    (zone_clearance 0.4)
     (zone_45_only no)
     (trace_min 0.2)
@@
     (visible_elements FFFFFF7F)
     (pcbplotparams
-      (layerselection 0x00030_80000001)
+      (layerselection 0x010f0_80000001)
       (usegerberextensions false)
       (excludeedgelayer true)
@@
       (plotvalue true)
       (plotinvisibletext false)
-      (padsonsilk false)
+      (padsonsilk true)
       (subtractmaskfromsilk false)
       (outputformat 1)
       (mirror false)
-      (drillshape 1)
+      (drillshape 0)
       (scaleselection 1)
       (outputdirectory /home/dariusz/Arduino/nrf24l01-net/pcb/sensor21/))
@@
     )
   )
+  (module Mounting_Holes:MountingHole_3mm (layer F.Cu)
+    (at 112.6 83.4)
+    (descr "Mounting hole, Befestigungsbohrung, 3mm, No Annular, Kein Restring,")
+    (tags "Mounting hole, Befestigungsbohrung, 3mm, No Annular, Kein Restring,")
+    (fp_text reference REF** (at 0 -4.0005) (layer F.SilkS) hide
+      (effects (font (size 1 1) (thickness 0.15)))
+    )
+    (fp_text value MountingHole_3mm (at 1.00076 5.00126) (layer F.Fab) hide
+      (effects (font (size 1 1) (thickness 0.15)))
+    )
+    (fp_circle (center 0 0) (end 3 0) (layer Cmts.User) (width 0.381))
+    (pad 1 thru_hole circle (at 0 0) (size 3 3) (drill 3) (layers))
+  )
+  (module Mounting_Holes:MountingHole_3mm (layer F.Cu)
+    (at 183.05 83.55)
+    (descr "Mounting hole, Befestigungsbohrung, 3mm, No Annular, Kein Restring,")
+    (tags "Mounting hole, Befestigungsbohrung, 3mm, No Annular, Kein Restring,")
+    (fp_text reference REF** (at 0 -4.0005) (layer F.SilkS) hide
+      (effects (font (size 1 1) (thickness 0.15)))
+    )
+    (fp_text value MountingHole_3mm (at 1.00076 5.00126) (layer F.Fab) hide
+      (effects (font (size 1 1) (thickness 0.15)))
+    )
+    (fp_circle (center 0 0) (end 3 0) (layer Cmts.User) (width 0.381))
+    (pad 1 thru_hole circle (at 0 0) (size 3 3) (drill 3) (layers))
+  )
+  (module Mounting_Holes:MountingHole_3mm (layer F.Cu)
+    (at 182.95 120.4)
+    (descr "Mounting hole, Befestigungsbohrung, 3mm, No Annular, Kein Restring,")
+    (tags "Mounting hole, Befestigungsbohrung, 3mm, No Annular, Kein Restring,")
+    (fp_text reference REF** (at 0 -4.0005) (layer F.SilkS) hide
+      (effects (font (size 1 1) (thickness 0.15)))
+    )
+    (fp_text value MountingHole_3mm (at 1.00076 5.00126) (layer F.Fab) hide
+      (effects (font (size 1 1) (thickness 0.15)))
+    )
+    (fp_circle (center 0 0) (end 3 0) (layer Cmts.User) (width 0.381))
+    (pad 1 thru_hole circle (at 0 0) (size 3 3) (drill 3) (layers))
+  )
+  (module Mounting_Holes:MountingHole_3mm (layer F.Cu)
+    (at 112.55 120.45)
+    (descr "Mounting hole, Befestigungsbohrung, 3mm, No Annular, Kein Restring,")
+    (tags "Mounting hole, Befestigungsbohrung, 3mm, No Annular, Kein Restring,")
+    (fp_text reference REF** (at 0 -4.0005) (layer F.SilkS) hide
+      (effects (font (size 1 1) (thickness 0.15)))
+    )
+    (fp_text value MountingHole_3mm (at 1.00076 5.00126) (layer F.Fab) hide
+      (effects (font (size 1 1) (thickness 0.15)))
+    )
+    (fp_circle (center 0 0) (end 3 0) (layer Cmts.User) (width 0.381))
+    (pad 1 thru_hole circle (at 0 0) (size 3 3) (drill 3) (layers))
+  )
   (gr_line (start 115.34 77.6) (end 115.44 77.6) (angle 90) (layer Edge.Cuts) (width 0.1))
-  (gr_line (start 115.34 124.39) (end 115.34 77.6) (angle 90) (layer Edge.Cuts) (width 0.1))
-  (gr_line (start 181.61 124.39) (end 115.34 124.39) (angle 90) (layer Edge.Cuts) (width 0.1))
-  (gr_line (start 181.61 77.6) (end 181.61 124.39) (angle 90) (layer Edge.Cuts) (width 0.1))
-  (gr_line (start 115.44 77.6) (end 181.61 77.6) (angle 90) (layer Edge.Cuts) (width 0.1))
+  (gr_line (start 107.74 125.64) (end 107.74 77.6) (angle 90) (layer Edge.Cuts) (width 0.1))
+  (gr_line (start 187.81 125.64) (end 107.74 125.64) (angle 90) (layer Edge.Cuts) (width 0.1))
+  (gr_line (start 187.81 77.6) (end 187.81 125.64) (angle 90) (layer Edge.Cuts) (width 0.1))
+  (gr_line (start 107.74 77.6) (end 187.81 77.6) (angle 90) (layer Edge.Cuts) (width 0.1))
   (segment (start 157.734 107.569) (end 157.76 107.57) (width 0.25) (layer F.Cu) (net 0) (status 80000))
   (segment (start 137.12 102.97) (end 132.57 102.97) (width 0.25) (layer B.Cu) (net 1))
@@
   (segment (start 122.27 106.99) (end 122.27 101.11) (width 0.25) (layer B.Cu) (net 27))
   (segment (start 122.27 101.11) (end 121.98 100.82) (width 0.25) (layer B.Cu) (net 27))
+  (zone (net 1) (net_name GND) (layer B.Cu) (hatch edge 0.508)
+    (connect_pads (clearance 0.4))
+    (min_thickness 0.2)
+    (fill yes (arc_segments 16) (thermal_gap 0.4) (thermal_bridge_width 0.29))
+    (polygon
+      (pts
+        (xy 187.25 124.9) (xy 108.3 124.95) (xy 108.3 78.1) (xy 187.25 78.1) (xy 187.25 124.9)
+      )
+    )
+  )
 )
