File: pcb/sensor21/sensor21.sch (KiCad schematic (older format))
At the start: 22 parts, among them IC1 ATMEGA8-P, P1 nRF24L01, P2 BME280, P3 CONN_01X02, Q1 BC548, U1 LM2931AZ-3.3/5.0, Y1 8Mhz

Commit message: all works ok
Parts:
- added C10, C9: 10u, Capacitors_ThroughHole:C_Radial_D5_L11_P2, symbol CP
- U1: value LM2931AZ-3.3/5.0 -> HT7333
Connections:
- net labels added: GNDPWR
- wire segments 89 -> 103
Changed lines of the file:
@@
 L GND #PWR09
 U 1 1 5A4F93BD
-P 7150 3100
-F 0 "#PWR09" H 7150 2850 50  0001 C CNN
-F 1 "GND" V 7050 3050 50  0000 C CNN
-F 2 "" H 7150 3100 50  0000 C CNN
-F 3 "" H 7150 3100 50  0000 C CNN
-	1    7150 3100
+P 6950 3100
+F 0 "#PWR09" H 6950 2850 50  0001 C CNN
+F 1 "GND" V 6850 3050 50  0000 C CNN
+F 2 "" H 6950 3100 50  0000 C CNN
+F 3 "" H 6950 3100 50  0000 C CNN
+	1    6950 3100
 	0    1    1    0
 $EndComp
@@
 P 3450 5750
 F 0 "U1" H 3450 6000 50  0000 C CNN
-F 1 "LM2931AZ-3.3/5.0" H 3450 5950 50  0000 C CNN
+F 1 "HT7333" H 3450 5950 50  0000 C CNN
 F 2 "TO_SOT_Packages_THT:TO-92_Inline_Narrow_Oval" H 3450 5850 50  0000 C CIN
 F 3 "" H 3450 5750 50  0000 C CNN
@@
 	-1   0    0    1
 $EndComp
+$Comp
+L CP C9
+U 1 1 5A74B5E4
+P 3000 5900
+F 0 "C9" H 3025 6000 50  0000 L CNN
+F 1 "10u" H 3025 5800 50  0000 L CNN
+F 2 "Capacitors_ThroughHole:C_Radial_D5_L11_P2" H 3038 5750 50  0001 C CNN
+F 3 "" H 3000 5900 50  0000 C CNN
+	1    3000 5900
+	1    0    0    -1
+$EndComp
+$Comp
+L CP C10
+U 1 1 5A74BCC2
+P 4000 5900
+F 0 "C10" H 4025 6000 50  0000 L CNN
+F 1 "10u" H 4025 5800 50  0000 L CNN
+F 2 "Capacitors_ThroughHole:C_Radial_D5_L11_P2" H 4038 5750 50  0001 C CNN
+F 3 "" H 4000 5900 50  0000 C CNN
+	1    4000 5900
+	1    0    0    -1
+$EndComp
+$Comp
+L GNDPWR #PWR018
+U 1 1 5A74C787
+P 6350 2500
+F 0 "#PWR018" H 6350 2300 50  0001 C CNN
+F 1 "GNDPWR" H 6350 2370 50  0000 C CNN
+F 2 "" H 6350 2450 50  0000 C CNN
+F 3 "" H 6350 2450 50  0000 C CNN
+	1    6350 2500
+	1    0    0    -1
+$EndComp
+$Comp
+L GNDPWR #PWR019
+U 1 1 5A74C9C3
+P 2800 5000
+F 0 "#PWR019" H 2800 4800 50  0001 C CNN
+F 1 "GNDPWR" H 2800 4870 50  0000 C CNN
+F 2 "" H 2800 4950 50  0000 C CNN
+F 3 "" H 2800 4950 50  0000 C CNN
+	1    2800 5000
+	1    0    0    -1
+$EndComp
+$Comp
+L GNDPWR #PWR020
+U 1 1 5A74CCBB
+P 6950 2850
+F 0 "#PWR020" H 6950 2650 50  0001 C CNN
+F 1 "GNDPWR" V 6850 2850 50  0000 C CNN
+F 2 "" H 6950 2800 50  0000 C CNN
+F 3 "" H 6950 2800 50  0000 C CNN
+	1    6950 2850
+	0    1    1    0
+$EndComp
+$Comp
+L GNDPWR #PWR021
+U 1 1 5A74CFA2
+P 4000 6300
+F 0 "#PWR021" H 4000 6100 50  0001 C CNN
+F 1 "GNDPWR" H 4000 6170 50  0000 C CNN
+F 2 "" H 4000 6250 50  0000 C CNN
+F 3 "" H 4000 6250 50  0000 C CNN
+	1    4000 6300
+	1    0    0    -1
+$EndComp
+$Comp
+L GNDPWR #PWR022
+U 1 1 5A74D1E6
+P 2000 2450
+F 0 "#PWR022" H 2000 2250 50  0001 C CNN
+F 1 "GNDPWR" H 2000 2320 50  0000 C CNN
+F 2 "" H 2000 2400 50  0000 C CNN
+F 3 "" H 2000 2400 50  0000 C CNN
+	1    2000 2450
+	1    0    0    -1
+$EndComp
+$Comp
+L GNDPWR #PWR023
+U 1 1 5A74D42B
+P 6300 4300
+F 0 "#PWR023" H 6300 4100 50  0001 C CNN
+F 1 "GNDPWR" H 6300 4170 50  0000 C CNN
+F 2 "" H 6300 4250 50  0000 C CNN
+F 3 "" H 6300 4250 50  0000 C CNN
+	1    6300 4300
+	1    0    0    -1
+$EndComp
 Wire Wire Line
 	2300 2650 1850 2650
@@
 	7450 5350 7450 5450
 Wire Wire Line
-	7100 5450 7100 5350
+	7100 5350 7100 5450
 Connection ~ 7100 5350
 Wire Wire Line
-	6650 5500 6650 5350
+	6650 5350 6650 5500
 Connection ~ 6650 5350
 Wire Wire Line
@@
 	7450 5850 7450 5750
 Wire Wire Line
-	7100 5750 7100 5850
+	7100 5850 7100 5750
 Connection ~ 7100 5850
 Wire Wire Line
-	6650 5700 6650 5850
+	6650 5850 6650 5700
 Connection ~ 6650 5850
 Wire Wire Line
@@
 	7850 3100 8050 3100
 Wire Wire Line
-	7150 3100 7350 3100
+	6950 3100 7350 3100
 Wire Wire Line
 	7450 2800 7250 2800
@@
 	5900 1600 5900 1500
 Wire Wire Line
-	5900 2450 5900 2300
+	5900 2300 5900 2450
 Wire Wire Line
 	5750 3550 5950 3550
@@
 	5850 5350 7450 5350
 Wire Wire Line
-	5850 5850 7450 5850
-Wire Wire Line
 	2800 5600 2800 6000
 Wire Wire Line
@@
 Connection ~ 2800 5700
 Wire Wire Line
-	2750 6100 3450 6100
+	2750 6100 4000 6100
 Connection ~ 3450 6100
 Wire Wire Line
@@
 Wire Wire Line
 	5850 5350 5850 5150
+Wire Wire Line
+	3000 5700 3000 5750
+Connection ~ 3000 5700
+Wire Wire Line
+	3000 6050 3000 6100
+Connection ~ 3000 6100
+Wire Wire Line
+	4000 5750 4000 5700
+Connection ~ 4000 5700
+Wire Wire Line
+	4000 6050 4000 6300
+Wire Wire Line
+	5900 2350 6350 2350
+Wire Wire Line
+	6350 2350 6350 2500
+Connection ~ 5900 2350
+Wire Wire Line
+	2800 4750 2800 5000
+Connection ~ 2800 4750
+Wire Wire Line
+	6950 2850 7100 2850
+Wire Wire Line
+	7100 2850 7100 3100
+Connection ~ 7100 3100
+Connection ~ 4000 6100
+Wire Wire Line
+	2000 2450 2000 2350
+Connection ~ 2000 2350
+Wire Wire Line
+	5950 4200 6300 4200
+Wire Wire Line
+	6300 4200 6300 4300
+$Comp
+L GNDPWR #PWR024
+U 1 1 5A74D73F
+P 6150 6000
+F 0 "#PWR024" H 6150 5800 50  0001 C CNN
+F 1 "GNDPWR" H 6150 5870 50  0000 C CNN
+F 2 "" H 6150 5950 50  0000 C CNN
+F 3 "" H 6150 5950 50  0000 C CNN
+	1    6150 6000
+	1    0    0    -1
+$EndComp
+Wire Wire Line
+	5850 5950 6150 5950
+Wire Wire Line
+	6150 5950 6150 6000
+Connection ~ 5850 5950
+Wire Wire Line
+	5850 5850 7450 5850
 $EndSCHEMATC

Commit message: all work well
Parts:
- removed U1: HT7333, TO_SOT_Packages_THT:TO-92_Inline_Narrow_Oval, symbol LM2931AZ-3.3/5.0
- added U1: HT7333, TO_SOT_Packages_THT:TO-92_Inline_Wide, symbol HT7333
- C2, C4, C5: footprint Capacitors_ThroughHole:C_Disc_D6_P5 -> Capacitors_ThroughHole:C_Disc_D3_P2.5
Connections:
- wire segments 103 -> 104
Changed lines of the file:
@@
 LIBS:valves
 LIBS:nRF24L01
+LIBS:HT7333
 LIBS:sensor21-cache
 EELAYER 25 0
@@
 F 0 "C2" V 2050 2050 50  0000 L CNN
 F 1 "100n" V 1950 2000 50  0000 L CNN
-F 2 "Capacitors_ThroughHole:C_Disc_D6_P5" H 2000 2250 50  0001 C CNN
+F 2 "Capacitors_ThroughHole:C_Disc_D3_P2.5" H 2000 2250 50  0001 C CNN
 F 3 "" H 2000 2250 50  0000 C CNN
 	1    2000 2250
@@
 F 0 "C4" H 6260 5670 50  0000 L CNN
 F 1 "100n" H 6260 5520 50  0000 L CNN
-F 2 "Capacitors_ThroughHole:C_Disc_D6_P5" H 6250 5600 50  0001 C CNN
+F 2 "Capacitors_ThroughHole:C_Disc_D3_P2.5" H 6250 5600 50  0001 C CNN
 F 3 "" H 6250 5600 50  0000 C CNN
 	1    6250 5600
@@
 F 0 "C5" H 6660 5670 50  0000 L CNN
 F 1 "100n" H 6660 5520 50  0000 L CNN
-F 2 "Capacitors_ThroughHole:C_Disc_D6_P5" H 6650 5600 50  0001 C CNN
+F 2 "Capacitors_ThroughHole:C_Disc_D3_P2.5" H 6650 5600 50  0001 C CNN
 F 3 "" H 6650 5600 50  0000 C CNN
 	1    6650 5600
@@
 NoConn ~ 4200 3450
 $Comp
-L LM2931AZ-3.3/5.0 U1
-U 1 1 5A4FEC87
-P 3450 5750
-F 0 "U1" H 3450 6000 50  0000 C CNN
-F 1 "HT7333" H 3450 5950 50  0000 C CNN
-F 2 "TO_SOT_Packages_THT:TO-92_Inline_Narrow_Oval" H 3450 5850 50  0000 C CIN
-F 3 "" H 3450 5750 50  0000 C CNN
-	1    3450 5750
-	1    0    0    -1
-$EndComp
-$Comp
 L +3.3V #PWR015
 U 1 1 5A4FED52
@@
 	7650 2200 8300 2200
 Wire Wire Line
-	8100 1450 8300 1450
+	8100 1450 8650 1450
 Wire Wire Line
 	8300 1450 8300 1200
@@
 Wire Wire Line
 	2800 5600 2800 6000
-Wire Wire Line
-	2800 5700 3050 5700
 Wire Wire Line
 	2800 6000 2750 6000
@@
 Wire Wire Line
 	5850 5850 7450 5850
+$Comp
+L HT7333 U1
+U 1 1 5A82B5D9
+P 3450 5700
+F 0 "U1" H 3450 5950 50  0000 C CNN
+F 1 "HT7333" H 3450 5900 50  0000 C CNN
+F 2 "TO_SOT_Packages_THT:TO-92_Inline_Wide" H 3450 5800 50  0000 C CIN
+F 3 "" H 3450 5700 50  0000 C CNN
+	1    3450 5700
+	1    0    0    -1
+$EndComp
+Wire Wire Line
+	2800 5700 3100 5700
+$Comp
+L PWR_FLAG #FLG025
+U 1 1 5A82B7CC
+P 8650 1250
+F 0 "#FLG025" H 8650 1345 50  0001 C CNN
+F 1 "PWR_FLAG" H 8650 1430 50  0000 C CNN
+F 2 "" H 8650 1250 50  0000 C CNN
+F 3 "" H 8650 1250 50  0000 C CNN
+	1    8650 1250
+	1    0    0    -1
+$EndComp
+Wire Wire Line
+	8650 1450 8650 1250
+Connection ~ 8300 1450
 $EndSCHEMATC

Commit message: some mesurements
Parts:
- added C11, C12: 100n, Capacitors_ThroughHole:C_Disc_D3_P2.5, symbol C
Connections:
- net +3V3: now also C12.1
- net GND: now also C11.2, C12.2
- net at C9.1, P3.2 (P2), U1.2 (VIN): now also C11.1
Other:
- moved on the sheet: P3
Changed lines of the file:
@@
 L +3.3V #PWR015
 U 1 1 5A4FED52
-P 4150 5700
-F 0 "#PWR015" H 4150 5550 50  0001 C CNN
-F 1 "+3.3V" H 4150 5840 50  0000 C CNN
-F 2 "" H 4150 5700 50  0000 C CNN
-F 3 "" H 4150 5700 50  0000 C CNN
-	1    4150 5700
+P 4650 5700
+F 0 "#PWR015" H 4650 5550 50  0001 C CNN
+F 1 "+3.3V" H 4650 5840 50  0000 C CNN
+F 2 "" H 4650 5700 50  0000 C CNN
+F 3 "" H 4650 5700 50  0000 C CNN
+	1    4650 5700
 	1    0    0    -1
 $EndComp
@@
 L PWR_FLAG #FLG017
 U 1 1 5A4FFD97
-P 2800 5600
-F 0 "#FLG017" H 2800 5695 50  0001 C CNN
-F 1 "PWR_FLAG" H 2800 5780 50  0000 C CNN
-F 2 "" H 2800 5600 50  0000 C CNN
-F 3 "" H 2800 5600 50  0000 C CNN
-	1    2800 5600
+P 2400 5600
+F 0 "#FLG017" H 2400 5695 50  0001 C CNN
+F 1 "PWR_FLAG" H 2400 5780 50  0000 C CNN
+F 2 "" H 2400 5600 50  0000 C CNN
+F 3 "" H 2400 5600 50  0000 C CNN
+	1    2400 5600
 	1    0    0    -1
 $EndComp
@@
 L CONN_01X02 P3
 U 1 1 5A50002A
-P 2550 6050
-F 0 "P3" H 2550 6200 50  0000 C CNN
-F 1 "CONN_01X02" V 2650 6050 50  0000 C CNN
-F 2 "Connect:GTK2400-V2" H 2550 6050 50  0001 C CNN
-F 3 "" H 2550 6050 50  0000 C CNN
-	1    2550 6050
+P 2150 6050
+F 0 "P3" H 2150 6200 50  0000 C CNN
+F 1 "CONN_01X02" V 2250 6050 50  0000 C CNN
+F 2 "Connect:GTK2400-V2" H 2150 6050 50  0001 C CNN
+F 3 "" H 2150 6050 50  0000 C CNN
+	1    2150 6050
 	-1   0    0    1
 $EndComp
@@
 Connection ~ 2250 4750
 Wire Wire Line
-	2300 2350 1650 2350
+	1650 2350 2300 2350
 Wire Wire Line
 	1650 2250 1650 4750
@@
 	2100 2250 2300 2250
 Wire Wire Line
-	3850 5700 4150 5700
+	3850 5700 4650 5700
 Wire Wire Line
 	3450 6000 3450 6250
@@
 	5850 5350 7450 5350
 Wire Wire Line
-	2800 5600 2800 6000
-Wire Wire Line
-	2800 6000 2750 6000
-Connection ~ 2800 5700
-Wire Wire Line
-	2750 6100 4000 6100
+	2400 5600 2400 6000
+Wire Wire Line
+	2400 6000 2350 6000
+Connection ~ 2400 5700
+Wire Wire Line
+	2350 6100 4350 6100
 Connection ~ 3450 6100
 Wire Wire Line
@@
 	1    0    0    -1
 $EndComp
-Wire Wire Line
-	2800 5700 3100 5700
 $Comp
 L PWR_FLAG #FLG025
@@
 	8650 1450 8650 1250
 Connection ~ 8300 1450
+$Comp
+L C C11
+U 1 1 5A8BF023
+P 2650 5900
+F 0 "C11" H 2675 6000 50  0000 L CNN
+F 1 "100n" H 2675 5800 50  0000 L CNN
+F 2 "Capacitors_ThroughHole:C_Disc_D3_P2.5" H 2688 5750 50  0001 C CNN
+F 3 "" H 2650 5900 50  0000 C CNN
+	1    2650 5900
+	1    0    0    -1
+$EndComp
+$Comp
+L C C12
+U 1 1 5A8BF0A3
+P 4350 5900
+F 0 "C12" H 4375 6000 50  0000 L CNN
+F 1 "100n" H 4375 5800 50  0000 L CNN
+F 2 "Capacitors_ThroughHole:C_Disc_D3_P2.5" H 4388 5750 50  0001 C CNN
+F 3 "" H 4350 5900 50  0000 C CNN
+	1    4350 5900
+	1    0    0    -1
+$EndComp
+Wire Wire Line
+	2400 5700 3100 5700
+Wire Wire Line
+	2650 5750 2650 5700
+Connection ~ 2650 5700
+Wire Wire Line
+	2650 6050 2650 6100
+Connection ~ 2650 6100
+Wire Wire Line
+	4350 6100 4350 6050
+Wire Wire Line
+	4350 5750 4350 5700
+Connection ~ 4350 5700
 $EndSCHEMATC

Commit message: wip
Parts:
- C1, C2, C3, C4, C5: symbol C_Small -> sensor21-rescue:C_Small
- C10, C6, C7, C8, C9: symbol CP -> sensor21-rescue:CP
- C11, C12: symbol C -> sensor21-rescue:C
- IC1: symbol ATMEGA8-P -> sensor21-rescue:ATMEGA8-P
- P1: symbol CONN_02X04 -> sensor21-rescue:CONN_02X04
- P2: symbol CONN_01X04 -> sensor21-rescue:CONN_01X04
- P3: symbol CONN_01X02 -> sensor21-rescue:CONN_01X02
- Q1: symbol BC548 -> sensor21-rescue:BC548
- R1, R2, R3, R5, R6, R7: symbol R -> sensor21-rescue:R
- R4: symbol Photores -> sensor21-rescue:Photores
- U1: symbol HT7333 -> HT7333:HT7333
- Y1: symbol Crystal -> sensor21-rescue:Crystal
